File: hardware/VoiceRecorder/VoiceRecorder.kicad_sch (KiCad schematic)
At the start: 10 parts, among them J1 Conn_01x03, J2 Micro_SD_Card, J3 Conn_01x03, J4 Conn_01x04, J5 Conn_01x03, J7 Conn_02x09_Counter_Clockwise, J8 Conn_01x03, SW1 SW_Push, SW2 SW_SPST

Commit message: finished pcb design
Parts:
- J1, J3, J5, J8: footprint (none) -> Connector_PinHeader_2.54mm:PinHeader_1x03_P2.54mm_Vertical
- J2: footprint (none) -> Connector_PinSocket_2.54mm:PinSocket_1x06_P2.54mm_Horizontal
- J4, J_1: footprint (none) -> Connector_PinHeader_2.54mm:PinHeader_1x04_P2.54mm_Vertical
- J7: footprint (none) -> footprints:ESP32-S3-SuperMini
- SW1: footprint (none) -> Button_Switch_THT:SW_Tactile_Straight_KSA0Axx1LFTR
- SW2: footprint (none) -> Connector_PinHeader_2.54mm:PinHeader_1x02_P2.54mm_Vertical
Connections:
- net +3.3V: now also J2.5 (VCC); no longer J2.4 (VDD)
- net GND: no longer J2.9 (SHIELD)
- net SD_CS: now also J2.1 (CS); no longer J2.2 (DAT3/CD)
- net SD_MISO: now also J2.4 (MISO); no longer J2.7 (DAT0)
- net SD_SCK: now also J2.2 (SCK); no longer J2.5 (CLK)
Other:
- moved on the sheet: J5
